File: hydrogen/board.sch (KiCad schematic (older format))
At the start: 38 parts, among them J1 Power, J10 OUT B3, J11 OUT B4, J2 IN A, J3 OUT A1, J4 OUT A2, J5 OUT A3, J6 OUT A4, J7 IN B, J8 OUT B1, J9 OUT B2, U1 OPA4991, U2 OPA4991, U3 LM358

Commit message: Rename folders
Parts:
- U3: footprint Package_SO:VSSOP-8_3.0x3.0mm_P0.65mm -> Package_SO:TSSOP-8_4.4x3mm_P0.65mm
Changed lines of the file:
@@
 Sheet 1 1
 Title "Hydrogen"
-Date "2021-10-02"
+Date "2021-10-07"
 Rev "v2"
 Comp "Winterbloom"
@@
 F 0 "U3" H 2550 5267 50  0000 C CNN
 F 1 "LM358" H 2550 5176 50  0000 C CNN
-F 2 "Package_SO:VSSOP-8_3.0x3.0mm_P0.65mm" H 2550 4900 50  0001 C CNN
+F 2 "Package_SO:TSSOP-8_4.4x3mm_P0.65mm" H 2550 4900 50  0001 C CNN
 F 3 "http://www.ti.com/lit/ds/symlink/lm2904-n.pdf" H 2550 4900 50  0001 C CNN
 F 4 "LM358DGKR" H 2550 4900 50  0001 C CNN "mpn"
@@
 F 0 "U3" H 6800 5267 50  0000 C CNN
 F 1 "LM358" H 6800 5176 50  0000 C CNN
-F 2 "Package_SO:VSSOP-8_3.0x3.0mm_P0.65mm" H 6800 4900 50  0001 C CNN
+F 2 "Package_SO:TSSOP-8_4.4x3mm_P0.65mm" H 6800 4900 50  0001 C CNN
 F 3 "http://www.ti.com/lit/ds/symlink/lm2904-n.pdf" H 6800 4900 50  0001 C CNN
 F 4 "LM358DGKR" H 6800 4900 50  0001 C CNN "mpn"
@@
 F 0 "U3" H 8508 5921 50  0000 L CNN
 F 1 "LM358" H 8508 5830 50  0000 L CNN
-F 2 "Package_SO:VSSOP-8_3.0x3.0mm_P0.65mm" H 8550 5875 50  0001 C CNN
+F 2 "Package_SO:TSSOP-8_4.4x3mm_P0.65mm" H 8550 5875 50  0001 C CNN
 F 3 "http://www.ti.com/lit/ds/symlink/lm2904-n.pdf" H 8550 5875 50  0001 C CNN
 F 4 "LM358DGKR" H 8550 5875 50  0001 C CNN "mpn"
@@
 Connection ~ 7075 4125
 $Comp
-L power:GND #PWR?
+L power:GND #PWR0125
 U 1 1 6159879A
 P 1225 1500
-F 0 "#PWR?" H 1225 1250 50  0001 C CNN
+F 0 "#PWR0125" H 1225 1250 50  0001 C CNN
 F 1 "GND" H 1230 1327 50  0000 C CNN
 F 2 "" H 1225 1500 50  0001 C CNN
