File: hydrogen/board.sch (KiCad schematic (older format))
At the start: 38 parts, among them J1 Power, J10 OUT B3, J11 OUT B4, J2 IN A, J3 OUT A1, J4 OUT A2, J5 OUT A3, J6 OUT A4, J7 IN B, J8 OUT B1, J9 OUT B2, U1 OPA4991, U2 OPA4991, U3 LM358

Commit message: Update hydrogen
Parts:
- D3, D5: Notes APT2012VBC/D -> Blue; mpn 151033BS03000 -> APT2012VBC/D
- D4, D6: Notes APT2012SURCK -> Red; mpn 151033RS03000 -> APT2012SURCK
- U3: mpn LM358DGKR -> LM358PWR
Changed lines of the file:
@@
 F 2 "Package_SO:TSSOP-8_4.4x3mm_P0.65mm" H 2550 4900 50  0001 C CNN
 F 3 "http://www.ti.com/lit/ds/symlink/lm2904-n.pdf" H 2550 4900 50  0001 C CNN
-F 4 "LM358DGKR" H 2550 4900 50  0001 C CNN "mpn"
+F 4 "LM358PWR" H 2550 4900 50  0001 C CNN "mpn"
 F 5 "" H 2550 4900 50  0001 C CNN "unit cost"
 	2    2550 4900
@@
 F 2 "winterbloom:LED_0805_Kingbright_APT2012" V 2975 5075 50  0001 C CNN
 F 3 "~" V 2975 5075 50  0001 C CNN
-F 4 "151033RS03000" H 2975 5075 50  0001 C CNN "mpn"
+F 4 "APT2012SURCK" H 2975 5075 50  0001 C CNN "mpn"
 F 5 "" H 2975 5075 50  0001 C CNN "unit cost"
-F 6 "APT2012SURCK" H 2975 5075 50  0001 C CNN "Notes"
+F 6 "Red" H 2975 5075 50  0001 C CNN "Notes"
 	1    2975 5075
 	0    1    1    0
@@
 F 2 "winterbloom:LED_0805_Kingbright_APT2012" V 2850 5075 50  0001 C CNN
 F 3 "~" V 2850 5075 50  0001 C CNN
-F 4 "151033BS03000" H 2850 5075 50  0001 C CNN "mpn"
+F 4 "APT2012VBC/D" H 2850 5075 50  0001 C CNN "mpn"
 F 5 "" H 2850 5075 50  0001 C CNN "unit cost"
-F 6 "APT2012VBC/D" H 2850 5075 50  0001 C CNN "Notes"
+F 6 "Blue" H 2850 5075 50  0001 C CNN "Notes"
 	1    2850 5075
 	0    -1   -1   0
@@
 F 2 "Package_SO:TSSOP-8_4.4x3mm_P0.65mm" H 6800 4900 50  0001 C CNN
 F 3 "http://www.ti.com/lit/ds/symlink/lm2904-n.pdf" H 6800 4900 50  0001 C CNN
-F 4 "LM358DGKR" H 6800 4900 50  0001 C CNN "mpn"
+F 4 "LM358PWR" H 6800 4900 50  0001 C CNN "mpn"
 F 5 "" H 6800 4900 50  0001 C CNN "unit cost"
 	1    6800 4900
@@
 F 2 "winterbloom:LED_0805_Kingbright_APT2012" V 7225 5075 50  0001 C CNN
 F 3 "~" V 7225 5075 50  0001 C CNN
-F 4 "151033RS03000" H 7225 5075 50  0001 C CNN "mpn"
+F 4 "APT2012SURCK" H 7225 5075 50  0001 C CNN "mpn"
 F 5 "" H 7225 5075 50  0001 C CNN "unit cost"
-F 6 "APT2012SURCK" H 7225 5075 50  0001 C CNN "Notes"
+F 6 "Red" H 7225 5075 50  0001 C CNN "Notes"
 	1    7225 5075
 	0    1    1    0
@@
 F 2 "winterbloom:LED_0805_Kingbright_APT2012" V 7100 5075 50  0001 C CNN
 F 3 "~" V 7100 5075 50  0001 C CNN
-F 4 "151033BS03000" H 7100 5075 50  0001 C CNN "mpn"
+F 4 "APT2012VBC/D" H 7100 5075 50  0001 C CNN "mpn"
 F 5 "" H 7100 5075 50  0001 C CNN "unit cost"
-F 6 "APT2012VBC/D" H 7100 5075 50  0001 C CNN "Notes"
+F 6 "Blue" H 7100 5075 50  0001 C CNN "Notes"
 	1    7100 5075
 	0    -1   -1   0
@@
 F 2 "Package_SO:TSSOP-8_4.4x3mm_P0.65mm" H 7825 6025 50  0001 C CNN
 F 3 "http://www.ti.com/lit/ds/symlink/lm2904-n.pdf" H 7825 6025 50  0001 C CNN
-F 4 "LM358DGKR" H 7825 6025 50  0001 C CNN "mpn"
+F 4 "LM358PWR" H 7825 6025 50  0001 C CNN "mpn"
 F 5 "" H 7825 6025 50  0001 C CNN "unit cost"
 	3    7825 6025
