File: helium/board.kicad_pcb (KiCad board)
At the start: 2 copper layers, 20 x 108 mm, 65 parts, among them J1 Power, J10 OUT B3, J12 IN C, J13 OUT C1, J14 OUT C2, J15 OUT C3, J17 OUT D, J18 IN D1, J19 IN D2, J2 IN A, J20 IN D3, J3 OUT A1, J4 OUT A2, J5 OUT A3, J7 IN B, J8 OUT B1, J9 OUT B2, U1 OPA4991, U2 OPA4991, U4 OPA4991, U6 OPA4991

Commit message: Add circle for QA sticker to Helium
Parts:
- added REF**: OSHW-Logo2_7.3x6mm_SilkScreen, Symbol:OSHW-Logo2_7.3x6mm_SilkScreen, B.Cu at (99.2, 80.7)
Other:
- board text added: "Helium v2 10/5/2021 CERN-OHL-P V2 helium.wntr.dev"
- board text removed: "CERN-OHL-P V2 helium.wntr.dev"
- board text removed: "Helium v2 10/5/2021"
